File: 03-led/board/kicad/03-led.kicad_sch (KiCad schematic)
At the start: 3 parts

Commit message: Update kicad projects
Connections:
- net at A1.5V1 (5V): now also R1.1; no longer R1.2
- net at A1.GND1 (GND): no longer D1.1 (K)
- net at D1.2 (A): now also R1.2; no longer R1.1
- new net GND: D1.1 (K)
Other:
- moved on the sheet: D1
Changed lines of the file:
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@@
 	(wire
 		(pts
-			(xy 127 48.26) (xy 121.92 48.26)
+			(xy 101.6 58.42) (xy 114.3 58.42)
 		)
 		(stroke
@@
 	(wire
 		(pts
-			(xy 127 49.53) (xy 127 48.26)
+			(xy 114.3 83.82) (xy 114.3 88.9)
 		)
 		(stroke
@@
 	(wire
 		(pts
-			(xy 101.6 58.42) (xy 127 58.42)
+			(xy 114.3 71.12) (xy 114.3 76.2)
 		)
 		(stroke
@@
 	(wire
 		(pts
-			(xy 101.6 48.26) (xy 114.3 48.26)
-		)
-		(stroke
-			(width 0)
-			(type default)
-		)
-	)
-	(wire
-		(pts
-			(xy 127 58.42) (xy 127 57.15)
+			(xy 114.3 58.42) (xy 114.3 63.5)
 		)
 		(stroke
@@
 	(symbol
 		(lib_id "Device:LED")
-		(at 118.11 48.26 0)
+		(at 114.3 80.01 90)
 		(unit 1)
 		(exclude_from_sim no)
@@
 		(fields_autoplaced yes)
 		(property "Reference" "D1"
-			(at 116.5225 41.91 0)
-			(effects
-				(font
-					(size 1.27 1.27)
-				)
+			(at 118.11 80.3274 90)
+			(effects
+				(font
+					(size 1.27 1.27)
+				)
+				(justify right)
 			)
 		)
 		(property "Value" "LED"
-			(at 116.5225 44.45 0)
-			(effects
-				(font
-					(size 1.27 1.27)
-				)
+			(at 118.11 82.8674 90)
+			(effects
+				(font
+					(size 1.27 1.27)
+				)
+				(justify right)
 			)
 		)
 		(property "Footprint" ""
-			(at 118.11 48.26 0)
+			(at 114.3 80.01 0)
 			(effects
 				(font
@@
 		)
 		(property "Datasheet" "~"
-			(at 118.11 48.26 0)
+			(at 114.3 80.01 0)
 			(effects
 				(font
@@
 		)
 		(property "Description" "Light emitting diode"
-			(at 118.11 48.26 0)
+			(at 114.3 80.01 0)
 			(effects
 				(font
@@
 		)
 		(property "Sim.Pins" "1=K 2=A"
-			(at 118.11 48.26 0)
+			(at 114.3 80.01 0)
 			(effects
 				(font
@@
 	(symbol
 		(lib_id "Device:R")
-		(at 127 53.34 0)
+		(at 114.3 67.31 0)
 		(unit 1)
 		(exclude_from_sim no)
@@
 		(fields_autoplaced yes)
 		(property "Reference" "R1"
-			(at 129.54 52.0699 0)
+			(at 116.84 66.0399 0)
 			(effects
 				(font
@@
 		)
 		(property "Value" "R"
-			(at 129.54 54.6099 0)
+			(at 116.84 68.5799 0)
 			(effects
 				(font
@@
 		)
 		(property "Footprint" ""
-			(at 125.222 53.34 90)
+			(at 112.522 67.31 90)
 			(effects
 				(font
@@
 		)
 		(property "Datasheet" "~"
-			(at 127 53.34 0)
+			(at 114.3 67.31 0)
 			(effects
 				(font
@@
 		)
 		(property "Description" "Resistor"
-			(at 127 53.34 0)
+			(at 114.3 67.31 0)
 			(effects
 				(font
@@
 					(unit 1)
 				)
+			)
+		)
+	)
+	(symbol
+		(lib_id "power:GND")
+		(at 114.3 88.9 0)
+		(unit 1)
+		(exclude_from_sim no)
+		(in_bom yes)
+		(on_board yes)
+		(dnp no)
+		(fields_autoplaced yes)
+		(property "Reference" "#PWR01"
+			(at 114.3 95.25 0)
+			(effects
+				(font
+					(size 1.27 1.27)
+				)
+				(hide yes)
+			)
+		)
+		(property "Value" "GND"
+			(at 114.3 93.98 0)
+			(effects
+				(font
+					(size 1.27 1.27)
+				)
+			)
+		)
+		(property "Footprint" ""
+			(at 114.3 88.9 0)
+			(effects
+				(font
+					(size 1.27 1.27)
+				)
+				(hide yes)
+			)
+		)
+		(property "Datasheet" ""
+			(at 114.3 88.9 0)
+			(effects
+				(font
+					(size 1.27 1.27)
+				)
+				(hide yes)
+			)
+		)
+		(property "Description" "Power symbol creates a global label with name \"GND\" , ground"
+			(at 114.3 88.9 0)
+			(effects
+				(font
+					(size 1.27 1.27)
+				)
+				(hide yes)
+			)
+		)
+		(pin "1"
+		)
+		(instances
+			(project ""
+				(path "/d8624d6d-7ef8-4e62-84c5-0e698729d9b8"
+					(reference "#PWR01")
+					(unit 1)
+				)
