File: 04-rgb-led/board/kicad/04-rgb-led.kicad_sch (KiCad schematic)
At the start: 5 parts

Commit message: Update kicad projects
Connections:
- net GND: now reaches D1.1 (RK), D1.2 (GK), D1.3 (BK)
- net GND: no longer A1.GND6 (GND)
Other:
- moved on the sheet: A1, D1, R1, R2, R3
