File: 05-digital-inputs/board/kicad/05-digital-inputs.kicad_sch (KiCad schematic)
At the start: 5 parts, among them SW1 SW_Push, SW2 SW_Push

Commit message: Update kicad projects
Connections:
- no-connect marks 0 -> 4
Other:
- moved on the sheet: A1, SW1
Changed lines of the file:
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@@
 	)
 	(junction
-		(at 139.7 52.07)
+		(at 139.7 54.61)
 		(diameter 0)
 		(color 0 0 0 0)
 	)
 	(junction
-		(at 149.86 52.07)
+		(at 149.86 54.61)
 		(diameter 0)
 		(color 0 0 0 0)
@@
 		(color 0 0 0 0)
 	)
+	(no_connect
+		(at 151.13 66.04)
+	)
+	(no_connect
+		(at 138.43 55.88)
+	)
+	(no_connect
+		(at 151.13 55.88)
+	)
+	(no_connect
+		(at 138.43 66.04)
+	)
 	(wire
 		(pts
@@
 	(wire
 		(pts
-			(xy 149.86 53.34) (xy 151.13 53.34)
+			(xy 149.86 55.88) (xy 151.13 55.88)
 		)
 		(stroke
@@
 	(wire
 		(pts
-			(xy 138.43 53.34) (xy 139.7 53.34)
+			(xy 138.43 55.88) (xy 139.7 55.88)
 		)
 		(stroke
@@
 	(wire
 		(pts
+			(xy 149.86 66.04) (xy 151.13 66.04)
+		)
+		(stroke
+			(width 0)
+			(type default)
+		)
+	)
+	(wire
+		(pts
 			(xy 149.86 64.77) (xy 149.86 66.04)
 		)
@@
 	(wire
 		(pts
-			(xy 127 50.8) (xy 139.7 50.8)
+			(xy 127 53.34) (xy 139.7 53.34)
 		)
 		(stroke
@@
 	(wire
 		(pts
-			(xy 139.7 52.07) (xy 139.7 53.34)
+			(xy 139.7 54.61) (xy 139.7 55.88)
 		)
 		(stroke
@@
 	(wire
 		(pts
-			(xy 149.86 52.07) (xy 149.86 50.8)
+			(xy 149.86 54.61) (xy 149.86 53.34)
 		)
 		(stroke
@@
 	(wire
 		(pts
-			(xy 127 50.8) (xy 127 57.15)
+			(xy 127 57.15) (xy 127 53.34)
 		)
 		(stroke
@@
 	(wire
 		(pts
-			(xy 177.8 114.3) (xy 177.8 50.8)
-		)
-		(stroke
-			(width 0)
-			(type default)
-		)
-	)
-	(wire
-		(pts
-			(xy 104.14 62.23) (xy 114.3 62.23)
-		)
-		(stroke
-			(width 0)
-			(type default)
-		)
-	)
-	(wire
-		(pts
-			(xy 149.86 52.07) (xy 149.86 53.34)
-		)
-		(stroke
-			(width 0)
-			(type default)
-		)
-	)
-	(wire
-		(pts
-			(xy 139.7 52.07) (xy 139.7 50.8)
-		)
-		(stroke
-			(width 0)
-			(type default)
-		)
-	)
-	(wire
-		(pts
-			(xy 104.14 57.15) (xy 127 57.15)
+			(xy 177.8 114.3) (xy 177.8 53.34)
+		)
+		(stroke
+			(width 0)
+			(type default)
+		)
+	)
+	(wire
+		(pts
+			(xy 101.6 62.23) (xy 114.3 62.23)
+		)
+		(stroke
+			(width 0)
+			(type default)
+		)
+	)
+	(wire
+		(pts
+			(xy 149.86 54.61) (xy 149.86 55.88)
+		)
+		(stroke
+			(width 0)
+			(type default)
+		)
+	)
+	(wire
+		(pts
+			(xy 139.7 54.61) (xy 139.7 53.34)
+		)
+		(stroke
+			(width 0)
+			(type default)
+		)
+	)
+	(wire
+		(pts
+			(xy 101.6 57.15) (xy 127 57.15)
 		)
 		(stroke
@@
 	(wire
 		(pts
-			(xy 149.86 50.8) (xy 177.8 50.8)
-		)
-		(stroke
-			(width 0)
-			(type default)
-		)
-	)
-	(wire
-		(pts
-			(xy 104.14 59.69) (xy 127 59.69)
+			(xy 149.86 53.34) (xy 177.8 53.34)
+		)
+		(stroke
+			(width 0)
+			(type default)
+		)
+	)
+	(wire
+		(pts
+			(xy 101.6 59.69) (xy 127 59.69)
 		)
 		(stroke
@@
 	(symbol
 		(lib_id "Switch:SW_Push")
-		(at 144.78 52.07 0)
+		(at 144.78 54.61 0)
 		(unit 1)
 		(exclude_from_sim no)
@@
 		(fields_autoplaced yes)
 		(property "Reference" "SW1"
-			(at 144.78 44.45 0)
+			(at 144.78 46.99 0)
 			(effects
 				(font
@@
 		)
 		(property "Value" "SW_Push"
-			(at 144.78 46.99 0)
+			(at 144.78 49.53 0)
 			(effects
 				(font
@@
 		)
 		(property "Footprint" ""
-			(at 144.78 46.99 0)
+			(at 144.78 49.53 0)
 			(effects
 				(font
@@
 		)
 		(property "Datasheet" "~"
-			(at 144.78 46.99 0)
+			(at 144.78 49.53 0)
 			(effects
 				(font
@@
 		)
 		(property "Description" "Push button switch, generic, two pins"
-			(at 144.78 52.07 0)
+			(at 144.78 54.61 0)
 			(effects
 				(font
@@
 	(symbol
 		(lib_id "PCM_arduino-library:Arduino_Mega2560_R3_Shield")
-		(at 71.12 104.14 0)
+		(at 68.58 104.14 0)
 		(unit 1)
 		(exclude_from_sim no)
@@
 		(fields_autoplaced yes)
 		(property "Reference" "A1"
-			(at 71.12 165.1 0)
+			(at 68.58 165.1 0)
 			(effects
 				(font
@@
 		)
 		(property "Value" "Arduino_Mega2560_R3_Shield"
-			(at 71.12 167.64 0)
+			(at 68.58 167.64 0)
 			(effects
 				(font
@@
 		)
 		(property "Footprint" "PCM_arduino-library:Arduino_Mega2560_R3_Shield"
-			(at 71.12 177.8 0)
+			(at 68.58 177.8 0)
 			(effects
 				(font
@@
 		)
 		(property "Datasheet" "https://docs.arduino.cc/hardware/mega-2560"
-			(at 71.12 173.99 0)
+			(at 68.58 173.99 0)
 			(effects
 				(font
@@
 		)
 		(property "Description" "Shield for Arduino Mega 2560 R3"
-			(at 71.12 104.14 0)
-			(effects
-				(font
+			(at 68.58 104.14 0)
+			(effects
+				(font
